File: m-brooks.kicad_pcb (KiCad board)
At the start: 2 copper layers, 101.6 x 50.8 mm, 18 parts, among them U2 LM336

Commit message: Trying to update to KiCAD v6
Parts:
- VADJ1: value R_POT -> 10k
Connections:
- BROOKS1 pad 0: Net-(BROOKS1-Pad0) -> unconnected-(BROOKS1-Pad0)
- BROOKS1 pad 13: (no net) -> unconnected-(BROOKS1-Pad13)
- BROOKS1 pad 14: (no net) -> unconnected-(BROOKS1-Pad14)
- BROOKS1 pad 15: (no net) -> unconnected-(BROOKS1-Pad15)
- BROOKS1 pad 3: (no net) -> unconnected-(BROOKS1-Pad3)
- BROOKS1 pad 6: (no net) -> unconnected-(BROOKS1-Pad6)
- BROOKS1 pad 8: (no net) -> unconnected-(BROOKS1-Pad8)
Other:
- net class Default removed
